Commit message: changed joint range for wrist joint

File: robot_model_config/urdf/ur5_model.urdf.xacro (robot description, xacro)
@@ -203,5 +203,5 @@
     <origin xyz="0.0 0.0 ${wrist_2_length}" rpy="0.0 0.0 0.0" />
     <axis xyz="0 1 0" />
-    <limit lower="${-1.5 * pi}" upper="${1.5 * pi}" effort="10.0" velocity="${pi}"/>
+    <limit lower="${-0.6 * pi}" upper="${0.6 * pi}" effort="10.0" velocity="${pi}"/>
     <dynamics damping="10" friction="0.1"/>
   </joint>
