Commit message: rotated arm base by 45 degrees

File: robot_model_config/urdf/ur5_2fgripper.xacro (robot description, xacro)
@@ -88,15 +88,7 @@
 			</collision>
 		</link>
-		<!--<link name="wrist_3_padding">
-			<collision>
-				<geometry>
-					<cylinder radius="0.10" length="0.12"/>
-				</geometry>
-				<material name="blue_transparent"/>
-			</collision>
-		</link>-->
 	<!-- sensor components -->
 		<xacro:sensor_definitions prefix="${arm_prefix}" parent_link="ur5_stand"
-			x_val="-0.981" y_val="0.190" z_val="1.015" pitch="1.145" yaw="0.035" roll="0.019" />
+			x_val="-1.20" y_val="0.190" z_val="1.015" pitch="1.145" yaw="0.035" roll="0.019" />
 	<!-- joints -->
 		<joint name="world_to_stand" type="fixed">
@@ -105,9 +97,4 @@
 			<origin xyz="-0.238 0 ${robot_stand_height * 0.5}"/>
 		</joint>
-		<!--<joint name="wrist_3_link_to_wrist_3_padding" type="fixed">
-			<parent link="wrist_3_link"/>
-			<child link="wrist_3_padding"/>
-			<origin xyz="0 0.09 0" rpy="1.57 0 0"/>
-		</joint>-->
 		<joint name="world_to_base_padding" type="fixed">
 			<parent link="world_frame"/>
@@ -118,5 +105,5 @@
 			<parent link="ur5_stand"/>
 			<child link="${arm_prefix}base_link"/>
-			<origin xyz="0 0 ${robot_stand_height * 0.5}" rpy="0 0 2.355"/>
+			<origin xyz="0 0 ${robot_stand_height * 0.5}" rpy="0 0 3.1416"/>
 		</joint>
 		<joint name="world_to_table" type="fixed">
@@ -128,5 +115,5 @@
 			<parent link="${arm_prefix}ee_link"/>
 			<child link="${arm_prefix}gripper_frame"/>
-			<origin xyz="0 0 0" rpy="-1.57 0 -1.57"/> <!-- 0 1.57 0 -->
+			<origin xyz="0 0 0" rpy="0 1.57 0"/> <!-- 0 1.57 0 -->
 		</joint>
 </robot>

Commit message: removed the table

File: robot_model_config/urdf/ur5_2fgripper.xacro (robot description, xacro)
@@ -64,5 +64,5 @@
 	<!-- workcell components -->
 		<link name="world_frame"/>
-		<xacro:work_table_link name="${arm_prefix}worktable" l="1.0" w="1.0" h="0.5"/>
+		<!--<xacro:work_table_link name="${arm_prefix}worktable" l="1.0" w="1.0" h="0.5"/>-->
 		<link name="ur5_stand">
 			<visual>
@@ -105,11 +105,11 @@
 			<parent link="ur5_stand"/>
 			<child link="${arm_prefix}base_link"/>
-			<origin xyz="0 0 ${robot_stand_height * 0.5}" rpy="0 0 3.1416"/>
+			<origin xyz="0 0 ${robot_stand_height * 0.5}" rpy="0 0 1.57"/>
 		</joint>
-		<joint name="world_to_table" type="fixed">
+		<!--<joint name="world_to_table" type="fixed">
 			<parent link="world_frame"/>
 			<child link="${arm_prefix}worktable"/>
 			<origin xyz="-1.02 0 0" rpy="0 0 0"/>
-		</joint>
+		</joint>-->
 		<joint name="${arm_prefix}to_gripper" type="fixed">
 			<parent link="${arm_prefix}ee_link"/>

Commit message: placed camera in the new location

File: robot_model_config/urdf/ur5_2fgripper.xacro (robot description, xacro)
@@ -90,5 +90,5 @@
 	<!-- sensor components -->
 		<xacro:sensor_definitions prefix="${arm_prefix}" parent_link="ur5_stand"
-			x_val="-1.20" y_val="0.190" z_val="1.015" pitch="1.145" yaw="0.035" roll="0.019" />
+			x_val="0.0" y_val="-0.810" z_val="0.6" roll="0.037" pitch="0.494" yaw="2.321" />
 	<!-- joints -->
 		<joint name="world_to_stand" type="fixed">
@@ -105,5 +105,5 @@
 			<parent link="ur5_stand"/>
 			<child link="${arm_prefix}base_link"/>
-			<origin xyz="0 0 ${robot_stand_height * 0.5}" rpy="0 0 1.57"/>
+			<origin xyz="0 0 ${robot_stand_height * 0.5}" rpy="0 0 -3.1415"/>
 		</joint>
 		<!--<joint name="world_to_table" type="fixed">

Commit message: added workcell walls

File: robot_model_config/urdf/ur5_2fgripper.xacro (robot description, xacro)
@@ -6,4 +6,7 @@
 	<!-- property list -->
 	<xacro:property name="workcell_height" value="1"/>
+	<xacro:property name="workcell_length" value="2.775"/>
+	<xacro:property name="workcell_width" value="2.220"/>
+	<xacro:property name="workcell_thickness" value="0.04"/>
 	<xacro:property name="robot_stand_height" value="0.20"/>
 	<xacro:property name="worktable_thickness" value="0.02"/>
@@ -15,4 +18,10 @@
 	<material name="yellow">
 		<color rgba="0 1 1 1"/>
+	</material>
+	<material name="gray_transparent">
+		<color rgba="0.6 0.6 0.6 0.4"/>
+	</material>
+	<material name="blue_transparent">
+		<color rgba="0 0.8 1 0.4"/>
 	</material>
 	<!-- instantiating arm and gripper -->
@@ -62,6 +71,60 @@
 			</link>
 		</xacro:macro>
+		<!-- geometry macros -->
+		<xacro:macro name="workcell_geometry" params="length width height *color_block">
+				<geometry>
+					<box size="${length} ${width} ${height}"/>
+				</geometry>
+				<xacro:insert_block name="color_block"/>
+		</xacro:macro>
+		<xacro:macro name="workcell_element" params="name parent length width height offset_x offset_y">
+			<link name="${name}">
+				<visual>
+					<xacro:workcell_geometry length="${length}" width="${width}" height="${height}">
+						<material name="gray_transparent"/>
+					</xacro:workcell_geometry>
+				</visual>
+				<collision>
+					<xacro:workcell_geometry length="${length}" width="${width}" height="${height}">
+						<material name="blue_transparent"/>
+					</xacro:workcell_geometry>
+				</collision>
+			</link>
+			<joint name="${parent}_to_${name}" type="fixed">
+				<parent link="${parent}"/>
+				<child link="${name}"/>
+				<origin xyz="${offset_x} ${offset_y} ${0.5 * height}" rpy="0 0 0"/>
+			</joint>
+		</xacro:macro>
+		<!-- end of geometry macros -->
+	<!-- workcell bounds macro -->
+		<xacro:macro name="workcell_bounds">
+			<link name="roof2">
+				<collision>
+					<origin xyz="0 0 ${workcell_height }" rpy="0 0 0"/>
+					<xacro:workcell_geometry length="${workcell_length * 0.5}"
+						 width="${workcell_width}" height="${workcell_thickness}">
+						<material name="blue_transparent"/>
+					</xacro:workcell_geometry>
+				</collision>
+			</link>
+			<joint name="workcell_to_roof2" type="fixed">
+				<parent link="world_frame"/>
+				<child link="roof2"/>
+				<origin xyz="${workcell_length * -0.25} 0 0" rpy="0 0 0"/>
+			</joint>
+			<xacro:workcell_element name="front_wall2" parent="world_frame"
+				 length="0.1" width="2.220" height="${workcell_height}" offset_x="-1.3375" offset_y="0"/>
+			<xacro:workcell_element name="back_wall2" parent="world_frame"
+				 length="0.04" width="2.00" height="${workcell_height}" offset_x="0.20" offset_y="0"/>
+			<xacro:workcell_element name="left_wall2" parent="world_frame"
+				length="1.384" width="0.1" height="${workcell_height}" offset_x="-0.601" offset_y="1.060"/>
+			<xacro:workcell_element name="right_wall2" parent="world_frame"
+				length="1.384" width="0.1" height="${workcell_height}" offset_x="-0.601" offset_y="-1.060"/>
+		</xacro:macro>
+	<!-- end of workcell bounds macro -->
 	<!-- workcell components -->
 		<link name="world_frame"/>
+		<xacro:workcell_bounds/>
 		<!--<xacro:work_table_link name="${arm_prefix}worktable" l="1.0" w="1.0" h="0.5"/>-->
 		<link name="ur5_stand">

Commit message: added alignment surface

File: robot_model_config/urdf/ur5_2fgripper.xacro (robot description, xacro)
@@ -128,4 +128,13 @@
 		<xacro:workcell_bounds/>
 		<!--<xacro:work_table_link name="${arm_prefix}worktable" l="1.0" w="1.0" h="0.5"/>-->
+		<link name="${arm_prefix}alignment_surface">
+			<visual>
+				<origin xyz="0 0 0" rpy="0 0 0"/>
+				<geometry>
+					<box size="1.2 1.2 0.01"/>
+				</geometry>
+				<material name="blue"/>
+			</visual>
+		</link>
 		<link name="ur5_stand">
 			<visual>
@@ -170,4 +179,9 @@
 			<origin xyz="0 0 ${robot_stand_height * 0.5}" rpy="0 0 -3.1415"/>
 		</joint>
+		<joint name="world_to_alignment_surface" type="fixed">
+			<parent link="world_frame"/>
+			<child link="${arm_prefix}alignment_surface"/>
+			<origin xyz="-1.20 0 0" rpy="0 0 0"/>
+		</joint>
 		<!--<joint name="world_to_table" type="fixed">
 			<parent link="world_frame"/>
