Commit message: added spacer

File: robot_model_config/urdf/simple_2fgripper_macro.xacro (robot description, xacro)
@@ -5,4 +5,6 @@
 	<xacro:property name="gripper_width" value="0.022"/>
 	<xacro:property name="gripper_height" value="0.08"/>
+	<xacro:property name="gripper_spacer_length" value="0.05"/>
+	<xacro:property name="gripper_spacer_radius" value="0.04"/>
 	<xacro:property name="finger_length" value="0.055"/>
 	<xacro:property name="finger_width" value="0.022"/>
@@ -45,4 +47,20 @@
 	<xacro:macro name="simple_2fgripper_link" params="prefix">
 		<link name="${prefix}gripper_frame"/>
+		<link name="${prefix}gripper_spacer">
+			<visual>
+				<origin xyz="0 0 0" rpy="0 0 0"/>
+				<geometry>
+					<cylinder length="${gripper_spacer_length}" radius="${gripper_spacer_radius}"/>
+				</geometry>
+				<material name="gray0"/>
+			</visual>
+			<collision>
+				<origin xyz="0 0 0" rpy="0 0 0"/>
+				<geometry>
+					<cylinder length="${gripper_spacer_length}" radius="${gripper_spacer_radius}"/>
+				</geometry>
+				<material name="gray0"/>
+			</collision>
+		</link>
 		<link name="${prefix}gripper_body">
 			<visual>
@@ -76,8 +94,13 @@
 			</collision>
 		</link>
+		<joint name="${prefix}gripper_frame_to_spacer" type="fixed">
+			<parent link="${prefix}gripper_frame"/>
+			<child link="${prefix}gripper_spacer"/>
+			<origin xyz="0 0 ${0.5*gripper_spacer_length}" rpy="0 0 0"/>
+		</joint>
 		<joint name="${prefix}gripper_frame_to_body" type="fixed">
 			<parent link="${prefix}gripper_frame"/>
 			<child link="${prefix}gripper_body"/>
-			<origin xyz="0 0 0" rpy="0 0 0"/>
+			<origin xyz="0 0 ${gripper_spacer_length}" rpy="0 0 0"/>
 		</joint>
 		<joint name="${prefix}gripper_to_tcp" type="fixed">

Commit message: increased lenght of the gripper

File: robot_model_config/urdf/simple_2fgripper_macro.xacro (robot description, xacro)
@@ -2,5 +2,5 @@
 <robot xmlns:xacro="http://ros.org/wiki/xacro">
 	<!-- parameter list -->
-	<xacro:property name="gripper_length" value="0.140"/>
+	<xacro:property name="gripper_length" value="0.150"/>
 	<xacro:property name="gripper_width" value="0.022"/>
 	<xacro:property name="gripper_height" value="0.08"/>
@@ -107,5 +107,5 @@
 			<parent link="${prefix}gripper_frame"/>
 			<child link="${prefix}tcp_frame"/>
-			<origin xyz=" 0 0 ${gripper_height + 0.6*finger_length}" rpy="0 0 0"/>
+			<origin xyz=" 0 0 ${gripper_height + gripper_spacer_length + 0.6*finger_length}" rpy="0 0 0"/>
 		</joint>
 	</xacro:macro>

Commit message: increased finger lenghts

File: robot_model_config/urdf/simple_2fgripper_macro.xacro (robot description, xacro)
@@ -7,5 +7,5 @@
 	<xacro:property name="gripper_spacer_length" value="0.05"/>
 	<xacro:property name="gripper_spacer_radius" value="0.04"/>
-	<xacro:property name="finger_length" value="0.055"/>
+	<xacro:property name="finger_length" value="0.065"/>
 	<xacro:property name="finger_width" value="0.022"/>
 	<xacro:property name="finger_thickness" value="0.008"/>

Commit message: increased the finger length and retreated the tcp position relative to the gripper body

File: robot_model_config/urdf/simple_2fgripper_macro.xacro (robot description, xacro)
@@ -7,5 +7,5 @@
 	<xacro:property name="gripper_spacer_length" value="0.05"/>
 	<xacro:property name="gripper_spacer_radius" value="0.04"/>
-	<xacro:property name="finger_length" value="0.065"/>
+	<xacro:property name="finger_length" value="0.07"/>
 	<xacro:property name="finger_width" value="0.022"/>
 	<xacro:property name="finger_thickness" value="0.008"/>
@@ -107,5 +107,5 @@
 			<parent link="${prefix}gripper_frame"/>
 			<child link="${prefix}tcp_frame"/>
-			<origin xyz=" 0 0 ${gripper_height + gripper_spacer_length + 0.6*finger_length}" rpy="0 0 0"/>
+			<origin xyz=" 0 0 ${gripper_height + gripper_spacer_length + 0.45*finger_length}" rpy="0 0 0"/>
 		</joint>
 	</xacro:macro>
